Commit message: add control system

File: sentinel_ws/src/sentry_description/urdf/chassis.xacro (robot description, xacro)
@@ -1,3157 +1,234 @@
 <?xml version='1.0' encoding='utf-8'?>
-<robot xmlns:xacro="http://www.ros.org/wiki/xacro">
-  <link name="base_link" />
+<!--
+  车体模型（纯 URDF，不含任何 Gazebo 内容）。
+  结构：base_link → chassis_link → 4 个全向轮 wheel_N_link → 每轮 28 个被动滚子 roller_NNN_link。
+  112 个滚子形状完全一致、只有位姿/轴线/质心/半径不同，因此统一由 cad_roller 宏生成；
+  注释里的数值全部来自 CAD 导出（tools/import_sentry_cad.py），不要手改。
+-->
+<robot name="robovigor_sentry" xmlns:xacro="http://www.ros.org/wiki/xacro">
+  <!-- ================= 常量区 ================= -->
+  <xacro:property name="cad_mesh" value="package://sentry_description/meshes"/>
+  <xacro:property name="roller_mass" value="0.00446428571429"/>
+  <xacro:property name="roller_effort" value="0.1"/>
+  <xacro:property name="roller_velocity" value="1000"/>
+  <xacro:property name="roller_damping" value="0.000001"/>
+  <xacro:property name="wheel_mass" value="0.25"/>
+  <xacro:property name="wheel_ixx" value="0.000251041666667"/>
+  <xacro:property name="wheel_izz" value="0.000189583333333"/>
+  <xacro:property name="wheel_radius" value="0.05"/>
+  <xacro:property name="wheel_length" value="0.04"/>
+  <!-- ================= 宏 ================= -->
+  <!-- 纯外观：CAD 网格 + 统一灰色材质（无 <color> 子元素，RViz 直接用默认色）。 -->
+  <xacro:macro name="cad_visual" params="file">
+    <visual>
+      <geometry>
+        <mesh filename="${cad_mesh}/${file}"/>
+      </geometry>
+      <material name="cad_gray"/>
+    </visual>
+  </xacro:macro>
+  <!-- 一个被动滚子 = 1 个 link + 1 个 continuous 关节。
+       碰撞体是包住滚子的球，惯量按球近似，球心/质心用 CAD 的 com。 -->
+  <xacro:macro name="cad_roller" params="id parent xyz axis com r i">
+    <link name="roller_${id}_link">
+      <xacro:cad_visual file="roller_${id}_link.stl"/>
+      <inertial>
+        <mass value="${roller_mass}"/>
+        <origin xyz="${com}"/>
+        <inertia ixx="${i}" iyy="${i}" izz="${i}" ixy="0" ixz="0" iyz="0"/>
+      </inertial>
+      <collision>
+        <geometry>
+          <sphere radius="${r}"/>
+        </geometry>
+        <origin xyz="${com}"/>
+      </collision>
+    </link>
+    <joint name="roller_${id}_joint" type="continuous">
+      <parent link="${parent}"/>
+      <child link="roller_${id}_link"/>
+      <origin xyz="${xyz}"/>
+      <axis xyz="${axis}"/>
+      <limit effort="${roller_effort}" velocity="${roller_velocity}"/>
+      <dynamics damping="${roller_damping}" friction="0"/>
+    </joint>
+  </xacro:macro>
+  <!-- 一个全向轮 = 1 个 link + 1 个 continuous 关节；碰撞体是包住轮子的圆柱。 -->
+  <xacro:macro name="cad_wheel" params="n xyz axis rpy ixy">
+    <link name="wheel_${n}_link">
+      <xacro:cad_visual file="wheel_${n}_link.stl"/>
+      <inertial>
+        <mass value="${wheel_mass}"/>
+        <inertia ixx="${wheel_ixx}" iyy="${wheel_ixx}" izz="${wheel_izz}"
+                 ixy="${ixy}" ixz="0" iyz="0"/>
+      </inertial>
+      <collision>
+        <geometry>
+          <cylinder radius="${wheel_radius}" length="${wheel_length}"/>
+        </geometry>
+        <origin xyz="0 0 0" rpy="${rpy}"/>
+      </collision>
+    </link>
+    <joint name="wheel_${n}_joint" type="continuous">
+      <parent link="chassis_link"/>
+      <child link="wheel_${n}_link"/>
+      <origin xyz="${xyz}"/>
+      <axis xyz="${axis}"/>
+      <limit effort="1.2" velocity="1000"/>
+      <dynamics damping="0.0001" friction="0"/>
+    </joint>
+  </xacro:macro>
+  <!-- ================= 车体（单个实例，直接写死） ================= -->
+  <link name="base_link"/>
+  <joint name="chassis_fixed" type="fixed">
+    <parent link="base_link"/>
+    <child link="chassis_link"/>
+  </joint>
   <link name="chassis_link">
     <visual>
       <geometry>
-        <mesh filename="package://sentry_description/meshes/chassis.stl" />
+        <mesh filename="${cad_mesh}/chassis.stl"/>
       </geometry>
       <material name="cad_gray">
-        <color rgba="0.48 0.51 0.55 1" />
+        <color rgba="0.48 0.51 0.55 1"/>
       </material>
     </visual>
     <collision>
-      <origin xyz="0 0 0" />
+      <origin xyz="0 0 0"/>
       <geometry>
-        <box size="0.30 0.30 0.08" />
+        <box size="0.30 0.30 0.08"/>
       </geometry>
     </collision>
     <inertial>
-      <origin xyz="0 0 -0.013000" />
-      <mass value="6.5" />
-      <inertia ixx="0.179616667" iyy="0.179616667" izz="0.3159" ixy="0" ixz="0" iyz="0" />
+      <origin xyz="0 0 -0.013000"/>
+      <mass value="6.5"/>
+      <inertia ixx="0.179616667" iyy="0.179616667" izz="0.3159" ixy="0" ixz="0" iyz="0"/>
     </inertial>
   </link>
-  <joint name="chassis_fixed" type="fixed">
-    <parent link="base_link" />
-    <child link="chassis_link" />
-  </joint>
-  <link name="roller_001_link">
-    <visual>
-      <geometry>
-        <mesh filename="package://sentry_description/meshes/roller_001_link.stl" />
-      </geometry>
-      <material name="cad_gray" />
-    </visual>
-    <inertial>
-      <mass value="0.00446428571429" />
-      <origin xyz="0.00599499324789 0.00599499324789 -0.00369900117728" />
-      <inertia ixx="1.75017872294e-07" iyy="1.75017872294e-07" izz="1.75017872294e-07" ixy="0" ixz="0" iyz="0" />
-    </inertial>
-    <collision>
-      <geometry>
-        <sphere radius="0.00990000042851228" />
-      </geometry>
-      <origin xyz="0.00599499324789 0.00599499324789 -0.00369900117728" />
-    </collision>
-  </link>
-  <joint name="roller_001_joint" type="continuous">
-    <parent link="wheel_1_link" />
-    <child link="roller_001_link" />
-    <origin xyz="-0.0328458544824 -0.0165823985151 -0.0569774201136" />
-    <axis xyz="0.648107386505 0.648107386505 -0.39989202432" />
-    <limit effort="0.1" velocity="1000" />
-    <dynamics damping="0.000001" friction="0" />
-  </joint>
-  <link name="roller_002_link">
-    <visual>
-      <geometry>
-        <mesh filename="package://sentry_description/meshes/roller_002_link.stl" />
-      </geometry>
-      <material name="cad_gray" />
-    </visual>
-    <inertial>
-      <mass value="0.00446428571429" />
-      <origin xyz="0.00653616373517 0.00653616373517 0.000345868542598" />
-      <inertia ixx="1.75017872293e-07" iyy="1.75017872293e-07" izz="1.75017872293e-07" ixy="0" ixz="0" iyz="0" />
-    </inertial>
-    <collision>
-      <geometry>
-        <sphere radius="0.009900000428501199" />
-      </geometry>
-      <origin xyz="0.00653616373517 0.00653616373517 0.000345868542598" />
-    </collision>
-  </link>
-  <joint name="roller_002_joint" type="continuous">
-    <parent link="wheel_1_link" />
-    <child link="roller_002_link" />
-    <origin xyz="-0.0129175924657 0.00334586350159 -0.066499575204" />
-    <axis xyz="0.7066123048 0.7066123048 0.0373911942762" />
-    <limit effort="0.1" velocity="1000" />
-    <dynamics damping="0.000001" friction="0" />
-  </joint>
-  <link name="roller_003_link">
-    <visual>
-      <geometry>
-        <mesh filename="package://sentry_description/meshes/roller_003_link.stl" />
-      </geometry>
-      <material name="cad_gray" />
-    </visual>
-    <inertial>
-      <mass value="0.00446428571429" />
-      <origin xyz="-0.00653616373516 -0.00653616373516 -0.000345868542597" />
-      <inertia ixx="1.75017872292e-07" iyy="1.75017872292e-07" izz="1.75017872292e-07" ixy="0" ixz="0" iyz="0" />
-    </inertial>
-    <collision>
-      <geometry>
-        <sphere radius="0.009900000428449006" />
-      </geometry>
-      <origin xyz="-0.00653616373516 -0.00653616373516 -0.000345868542597" />
-    </collision>
-  </link>
-  <joint name="roller_003_joint" type="continuous">
-    <parent link="wheel_1_link" />
-    <child link="roller_003_link" />
-    <origin xyz="-0.00334586350159 0.0129175924657 0.066499575204" />
-    <axis xyz="-0.7066123048 -0.7066123048 -0.0373911942762" />
-    <limit effort="0.1" velocity="1000" />
-    <dynamics damping="0.000001" friction="0" />
-  </joint>
-  <link name="roller_004_link">
-    <visual>
-      <geometry>
-        <mesh filename="package://sentry_description/meshes/roller_004_link.stl" />
-      </geometry>
-      <material name="cad_gray" />
-    </visual>
-    <inertial>
-      <mass value="0.00446428571429" />
-      <origin xyz="-0.00599499324791 -0.00599499324791 0.00369900117729" />
-      <inertia ixx="1.75017872292e-07" iyy="1.75017872292e-07" izz="1.75017872292e-07" ixy="0" ixz="0" iyz="0" />
-    </inertial>
-    <collision>
-      <geometry>
-        <sphere radius="0.009900000428462149" />
-      </geometry>
-      <origin xyz="-0.00599499324791 -0.00599499324791 0.00369900117729" />
-    </collision>
-  </link>
-  <joint name="roller_004_joint" type="continuous">
-    <parent link="wheel_1_link" />
-    <child link="roller_004_link" />
-    <origin xyz="0.0165823985151 0.0328458544824 0.0569774201136" />
-    <axis xyz="-0.648107386505 -0.648107386505 0.39989202432" />
-    <limit effort="0.1" velocity="1000" />
-    <dynamics damping="0.000001" friction="0" />
-  </joint>
-  <link name="roller_005_link">
-    <visual>
-      <geometry>
-        <mesh filename="package://sentry_description/meshes/roller_005_link.stl" />
-      </geometry>
-      <material name="cad_gray" />
-    </visual>
-    <inertial>
-      <mass value="0.00446428571429" />
-      <origin xyz="0.00169286747068 0.00169286747068 -0.00893481377798" />
-      <inertia ixx="1.75017872294e-07" iyy="1.75017872294e-07" izz="1.75017872294e-07" ixy="0" ixz="0" iyz="0" />
-    </inertial>
-    <collision>
-      <geometry>
-        <sphere radius="0.009900000428507517" />
-      </geometry>
-      <origin xyz="0.00169286747068 0.00169286747068 -0.00893481377798" />
-    </collision>
-  </link>
-  <joint name="roller_005_joint" type="continuous">
-    <parent link="wheel_1_link" />
-    <child link="roller_005_link" />
-    <origin xyz="-0.0550400363414 -0.0387765803741 -0.00819900689261" />
-    <axis xyz="0.183012701892 0.183012701892 -0.965925826289" />
-    <limit effort="0.1" velocity="1000" />
-    <dynamics damping="0.000001" friction="0" />
-  </joint>
-  <link name="roller_006_link">
-    <visual>
-      <geometry>
-        <mesh filename="package://sentry_description/meshes/roller_006_link.stl" />
-      </geometry>
-      <material name="cad_gray" />
-    </visual>
-    <inertial>
-      <mass value="0.00446428571429" />
-      <origin xyz="0.001215999047 0.001215999047 0.00908873976031" />
-      <inertia ixx="1.75017872292e-07" iyy="1.75017872292e-07" izz="1.75017872292e-07" ixy="0" ixz="0" iyz="0" />
-    </inertial>
-    <collision>
-      <geometry>
-        <sphere radius="0.00990000042846859" />
-      </geometry>
-      <origin xyz="0.001215999047 0.001215999047 0.00908873976031" />
-    </collision>
-  </link>
-  <joint name="roller_006_joint" type="continuous">
-    <parent link="wheel_1_link" />
-    <child link="roller_006_link" />
-    <origin xyz="0.0366466703055 0.0529101262727 -0.0213960882716" />
-    <axis xyz="0.131459358126 0.131459358126 0.982566473233" />
-    <limit effort="0.1" velocity="1000" />
-    <dynamics damping="0.000001" friction="0" />
-  </joint>
-  <link name="roller_007_link">
-    <visual>
-      <geometry>
-        <mesh filename="package://sentry_description/meshes/roller_007_link.stl" />
-      </geometry>
-      <material name="cad_gray" />
-    </visual>
-    <inertial>
-      <mass value="0.00446428571429" />
-      <origin xyz="-0.00578276683385 -0.00578276683385 -0.00432223475579" />
-      <inertia ixx="1.75017872294e-07" iyy="1.75017872294e-07" izz="1.75017872294e-07" ixy="0" ixz="0" iyz="0" />
-    </inertial>
-    <collision>
-      <geometry>
-        <sphere radius="0.009900000428505635" />
-      </geometry>
-      <origin xyz="-0.00578276683385 -0.00578276683385 -0.00432223475579" />
-    </collision>
-  </link>
-  <joint name="roller_007_joint" type="continuous">
-    <parent link="wheel_1_link" />
-    <child link="roller_007_link" />
-    <origin xyz="-0.0242220246738 -0.00795856870646 0.0628506738615" />
-    <axis xyz="-0.625163990099 -0.625163990099 -0.467268628273" />
-    <limit effort="0.1" velocity="1000" />
-    <dynamics damping="0.000001" friction="0" />
-  </joint>
-  <link name="roller_008_link">
-    <visual>
-      <geometry>
-        <mesh filename="package://sentry_description/meshes/roller_008_link.stl" />
-      </geometry>
-      <material name="cad_gray" />
-    </visual>
-    <inertial>
-      <mass value="0.00446428571429" />
-      <origin xyz="0.00578276683391 0.00578276683391 0.00432223475584" />
-      <inertia ixx="1.75017872293e-07" iyy="1.75017872293e-07" izz="1.75017872293e-07" ixy="0" ixz="0" iyz="0" />
-    </inertial>
-    <collision>
-      <geometry>
-        <sphere radius="0.009900000428476167" />
-      </geometry>
-      <origin xyz="0.00578276683391 0.00578276683391 0.00432223475584" />
-    </collision>
-  </link>
-  <joint name="roller_008_joint" type="continuous">
-    <parent link="wheel_1_link" />
-    <child link="roller_008_link" />
-    <origin xyz="0.00795856870646 0.0242220246737 -0.0628506738615" />
-    <axis xyz="0.625163990099 0.625163990099 0.467268628273" />
-    <limit effort="0.1" velocity="1000" />
-    <dynamics damping="0.000001" friction="0" />
-  </joint>
-  <link name="roller_009_link">
-    <visual>
-      <geometry>
-        <mesh filename="package://sentry_description/meshes/roller_009_link.stl" />
-      </geometry>
-      <material name="cad_gray" />
-    </visual>
-    <inertial>
-      <mass value="0.00446428571429" />
-      <origin xyz="0.00388402204018 0.00388402204018 0.00744252936694" />
-      <inertia ixx="1.75017872294e-07" iyy="1.75017872294e-07" izz="1.75017872294e-07" ixy="0" ixz="0" iyz="0" />
-    </inertial>
-    <collision>
-      <geometry>
-        <sphere radius="0.00990000042852242" />
-      </geometry>
-      <origin xyz="0.00388402204018 0.00388402204018 0.00744252936694" />
-    </collision>
-  </link>
-  <joint name="roller_009_joint" type="continuous">
-    <parent link="wheel_1_link" />
-    <child link="roller_009_link" />
-    <origin xyz="0.0256478492846 0.0419113052519 -0.0467534257478" />
-    <axis xyz="0.419894280025 0.419894280025 0.804597779766" />
-    <limit effort="0.1" velocity="1000" />
-    <dynamics damping="0.000001" friction="0" />
-  </joint>
-  <link name="roller_010_link">
-    <visual>
-      <geometry>
-        <mesh filename="package://sentry_description/meshes/roller_010_link.stl" />
-      </geometry>
-      <material name="cad_gray" />
-    </visual>
-    <inertial>
-      <mass value="0.00446428571429" />
-      <origin xyz="-0.00169286747069 -0.00169286747069 0.00893481377805" />
-      <inertia ixx="1.75017872293e-07" iyy="1.75017872293e-07" izz="1.75017872293e-07" ixy="0" ixz="0" iyz="0" />
-    </inertial>
-    <collision>
-      <geometry>
-        <sphere radius="0.009900000428488924" />
-      </geometry>
-      <origin xyz="-0.00169286747069 -0.00169286747069 0.00893481377805" />
-    </collision>
-  </link>
-  <joint name="roller_010_joint" type="continuous">
-    <parent link="wheel_1_link" />
-    <child link="roller_010_link" />
-    <origin xyz="0.0387765803741 0.0550400363414 0.00819900689261" />
-    <axis xyz="-0.183012701892 -0.183012701892 0.965925826289" />
-    <limit effort="0.1" velocity="1000" />
-    <dynamics damping="0.000001" friction="0" />
-  </joint>
-  <link name="roller_011_link">
-    <visual>
-      <geometry>
-        <mesh filename="package://sentry_description/meshes/roller_011_link.stl" />
-      </geometry>
-      <material name="cad_gray" />
-    </visual>
-    <inertial>
-      <mass value="0.00446428571429" />
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