Commit message: add control system

File: sentinel_ws/src/sentry_sim/urdf/sentry_sim.urdf.xacro (robot description, xacro)
@@ -1,11 +1,36 @@
 <?xml version='1.0' encoding='utf-8'?>
+<!--
+  Gazebo Classic 专用外壳：引用纯模型，再追加材质、接触参数与两个自写插件。
+  纯 RViz 看模型时不要用这个文件，用 sentry_description/urdf/sentry.urdf.xacro。
+-->
 <robot name="robovigor_sentry" xmlns:xacro="http://www.ros.org/wiki/xacro">
-  <xacro:include filename="$(find sentry_description)/urdf/sentry.urdf.xacro" />
-  <gazebo reference="chassis_link">
-    <material>Gazebo/Grey</material>
-  </gazebo>
-  <gazebo reference="gimbal_yaw_link">
-    <material>Gazebo/Grey</material>
-  </gazebo>
+  <xacro:include filename="$(find sentry_description)/urdf/sentry.urdf.xacro"/>
+  <!-- 所有零件统一灰色，避免 Gazebo 给每个网格随机配色 -->
+  <xacro:macro name="gazebo_grey" params="link">
+    <gazebo reference="${link}">
+      <material>Gazebo/Grey</material>
+    </gazebo>
+  </xacro:macro>
+  <!-- 滚子接触参数：高刚度 + 软阻尼，压住全向轮打滑 -->
+  <xacro:macro name="roller_surface" params="n">
+    <gazebo reference="roller_${n}_link">
+      <material>Gazebo/Grey</material>
+      <mu1>0.9</mu1>
+      <mu2>0.9</mu2>
+      <kp>100000</kp>
+      <kd>100</kd>
+      <minDepth>0.00005</minDepth>
+      <maxVel>0.1</maxVel>
+      <maxContacts>3</maxContacts>
+    </gazebo>
+  </xacro:macro>
+  <xacro:gazebo_grey link="chassis_link"/>
+  <xacro:gazebo_grey link="gimbal_yaw_link"/>
+  <xacro:gazebo_grey link="wheel_1_link"/>
+  <xacro:gazebo_grey link="wheel_2_link"/>
+  <xacro:gazebo_grey link="wheel_3_link"/>
+  <xacro:gazebo_grey link="wheel_4_link"/>
+  <!-- 两个自写插件挂在同一个 <gazebo> 下：
+       云台力矩稳定（收 /spin_mode，发 /gimbal_pose）+ 四轮力矩驱动（/odom、/joint_states）。 -->
   <gazebo>
     <plugin name="sentry_gimbal_stabilizer" filename="libsentry_gimbal_stabilizer.so">
@@ -32,1135 +57,120 @@
     </plugin>
   </gazebo>
-  <gazebo reference="roller_001_link">
-    <material>Gazebo/Grey</material>
-    <mu1>0.9</mu1>
-    <mu2>0.9</mu2>
-    <kp>100000</kp>
-    <kd>100</kd>
-    <minDepth>0.00005</minDepth>
-    <maxVel>0.1</maxVel>
-    <maxContacts>3</maxContacts>
-  </gazebo>
-  <gazebo reference="roller_002_link">
-    <material>Gazebo/Grey</material>
-    <mu1>0.9</mu1>
-    <mu2>0.9</mu2>
-    <kp>100000</kp>
-    <kd>100</kd>
-    <minDepth>0.00005</minDepth>
-    <maxVel>0.1</maxVel>
-    <maxContacts>3</maxContacts>
-  </gazebo>
-  <gazebo reference="roller_003_link">
-    <material>Gazebo/Grey</material>
-    <mu1>0.9</mu1>
-    <mu2>0.9</mu2>
-    <kp>100000</kp>
-    <kd>100</kd>
-    <minDepth>0.00005</minDepth>
-    <maxVel>0.1</maxVel>
-    <maxContacts>3</maxContacts>
-  </gazebo>
-  <gazebo reference="roller_004_link">
-    <material>Gazebo/Grey</material>
-    <mu1>0.9</mu1>
-    <mu2>0.9</mu2>
-    <kp>100000</kp>
-    <kd>100</kd>
-    <minDepth>0.00005</minDepth>
-    <maxVel>0.1</maxVel>
-    <maxContacts>3</maxContacts>
-  </gazebo>
-  <gazebo reference="roller_005_link">
-    <material>Gazebo/Grey</material>
-    <mu1>0.9</mu1>
-    <mu2>0.9</mu2>
-    <kp>100000</kp>
-    <kd>100</kd>
-    <minDepth>0.00005</minDepth>
-    <maxVel>0.1</maxVel>
-    <maxContacts>3</maxContacts>
-  </gazebo>
-  <gazebo reference="roller_006_link">
-    <material>Gazebo/Grey</material>
-    <mu1>0.9</mu1>
-    <mu2>0.9</mu2>
-    <kp>100000</kp>
-    <kd>100</kd>
-    <minDepth>0.00005</minDepth>
-    <maxVel>0.1</maxVel>
-    <maxContacts>3</maxContacts>
-  </gazebo>
-  <gazebo reference="roller_007_link">
-    <material>Gazebo/Grey</material>
-    <mu1>0.9</mu1>
-    <mu2>0.9</mu2>
-    <kp>100000</kp>
-    <kd>100</kd>
-    <minDepth>0.00005</minDepth>
-    <maxVel>0.1</maxVel>
-    <maxContacts>3</maxContacts>
-  </gazebo>
-  <gazebo reference="roller_008_link">
-    <material>Gazebo/Grey</material>
-    <mu1>0.9</mu1>
-    <mu2>0.9</mu2>
-    <kp>100000</kp>
-    <kd>100</kd>
-    <minDepth>0.00005</minDepth>
-    <maxVel>0.1</maxVel>
-    <maxContacts>3</maxContacts>
-  </gazebo>
-  <gazebo reference="roller_009_link">
-    <material>Gazebo/Grey</material>
-    <mu1>0.9</mu1>
-    <mu2>0.9</mu2>
-    <kp>100000</kp>
-    <kd>100</kd>
-    <minDepth>0.00005</minDepth>
-    <maxVel>0.1</maxVel>
-    <maxContacts>3</maxContacts>
-  </gazebo>
-  <gazebo reference="roller_010_link">
-    <material>Gazebo/Grey</material>
-    <mu1>0.9</mu1>
-    <mu2>0.9</mu2>
-    <kp>100000</kp>
-    <kd>100</kd>
-    <minDepth>0.00005</minDepth>
-    <maxVel>0.1</maxVel>
-    <maxContacts>3</maxContacts>
-  </gazebo>
-  <gazebo reference="roller_011_link">
-    <material>Gazebo/Grey</material>
-    <mu1>0.9</mu1>
-    <mu2>0.9</mu2>
-    <kp>100000</kp>
-    <kd>100</kd>
-    <minDepth>0.00005</minDepth>
-    <maxVel>0.1</maxVel>
-    <maxContacts>3</maxContacts>
-  </gazebo>
-  <gazebo reference="roller_012_link">
-    <material>Gazebo/Grey</material>
-    <mu1>0.9</mu1>
-    <mu2>0.9</mu2>
-    <kp>100000</kp>
-    <kd>100</kd>
-    <minDepth>0.00005</minDepth>
-    <maxVel>0.1</maxVel>
-    <maxContacts>3</maxContacts>
-  </gazebo>
-  <gazebo reference="roller_013_link">
-    <material>Gazebo/Grey</material>
-    <mu1>0.9</mu1>
-    <mu2>0.9</mu2>
-    <kp>100000</kp>
-    <kd>100</kd>
-    <minDepth>0.00005</minDepth>
-    <maxVel>0.1</maxVel>
-    <maxContacts>3</maxContacts>
-  </gazebo>
-  <gazebo reference="roller_014_link">
-    <material>Gazebo/Grey</material>
-    <mu1>0.9</mu1>
-    <mu2>0.9</mu2>
-    <kp>100000</kp>
-    <kd>100</kd>
-    <minDepth>0.00005</minDepth>
-    <maxVel>0.1</maxVel>
-    <maxContacts>3</maxContacts>
-  </gazebo>
-  <gazebo reference="roller_015_link">
-    <material>Gazebo/Grey</material>
-    <mu1>0.9</mu1>
-    <mu2>0.9</mu2>
-    <kp>100000</kp>
-    <kd>100</kd>
-    <minDepth>0.00005</minDepth>
-    <maxVel>0.1</maxVel>
-    <maxContacts>3</maxContacts>
-  </gazebo>
-  <gazebo reference="roller_016_link">
-    <material>Gazebo/Grey</material>
-    <mu1>0.9</mu1>
-    <mu2>0.9</mu2>
-    <kp>100000</kp>
-    <kd>100</kd>
-    <minDepth>0.00005</minDepth>
-    <maxVel>0.1</maxVel>
-    <maxContacts>3</maxContacts>
-  </gazebo>
-  <gazebo reference="roller_017_link">
-    <material>Gazebo/Grey</material>
-    <mu1>0.9</mu1>
-    <mu2>0.9</mu2>
-    <kp>100000</kp>
-    <kd>100</kd>
-    <minDepth>0.00005</minDepth>
-    <maxVel>0.1</maxVel>
-    <maxContacts>3</maxContacts>
-  </gazebo>
-  <gazebo reference="roller_018_link">
-    <material>Gazebo/Grey</material>
-    <mu1>0.9</mu1>
-    <mu2>0.9</mu2>
-    <kp>100000</kp>
-    <kd>100</kd>
-    <minDepth>0.00005</minDepth>
-    <maxVel>0.1</maxVel>
-    <maxContacts>3</maxContacts>
-  </gazebo>
-  <gazebo reference="roller_019_link">
-    <material>Gazebo/Grey</material>
-    <mu1>0.9</mu1>
-    <mu2>0.9</mu2>
-    <kp>100000</kp>
-    <kd>100</kd>
-    <minDepth>0.00005</minDepth>
-    <maxVel>0.1</maxVel>
-    <maxContacts>3</maxContacts>
-  </gazebo>
-  <gazebo reference="roller_020_link">
-    <material>Gazebo/Grey</material>
-    <mu1>0.9</mu1>
-    <mu2>0.9</mu2>
-    <kp>100000</kp>
-    <kd>100</kd>
-    <minDepth>0.00005</minDepth>
-    <maxVel>0.1</maxVel>
-    <maxContacts>3</maxContacts>
-  </gazebo>
-  <gazebo reference="roller_021_link">
-    <material>Gazebo/Grey</material>
-    <mu1>0.9</mu1>
-    <mu2>0.9</mu2>
-    <kp>100000</kp>
-    <kd>100</kd>
-    <minDepth>0.00005</minDepth>
-    <maxVel>0.1</maxVel>
-    <maxContacts>3</maxContacts>
-  </gazebo>
-  <gazebo reference="roller_022_link">
-    <material>Gazebo/Grey</material>
-    <mu1>0.9</mu1>
-    <mu2>0.9</mu2>
-    <kp>100000</kp>
-    <kd>100</kd>
-    <minDepth>0.00005</minDepth>
-    <maxVel>0.1</maxVel>
-    <maxContacts>3</maxContacts>
-  </gazebo>
-  <gazebo reference="roller_023_link">
-    <material>Gazebo/Grey</material>
-    <mu1>0.9</mu1>
-    <mu2>0.9</mu2>
-    <kp>100000</kp>
-    <kd>100</kd>
-    <minDepth>0.00005</minDepth>
-    <maxVel>0.1</maxVel>
-    <maxContacts>3</maxContacts>
-  </gazebo>
-  <gazebo reference="roller_024_link">
-    <material>Gazebo/Grey</material>
-    <mu1>0.9</mu1>
-    <mu2>0.9</mu2>
-    <kp>100000</kp>
-    <kd>100</kd>
-    <minDepth>0.00005</minDepth>
-    <maxVel>0.1</maxVel>
-    <maxContacts>3</maxContacts>
-  </gazebo>
-  <gazebo reference="roller_025_link">
-    <material>Gazebo/Grey</material>
-    <mu1>0.9</mu1>
-    <mu2>0.9</mu2>
-    <kp>100000</kp>
-    <kd>100</kd>
-    <minDepth>0.00005</minDepth>
-    <maxVel>0.1</maxVel>
-    <maxContacts>3</maxContacts>
-  </gazebo>
-  <gazebo reference="roller_026_link">
-    <material>Gazebo/Grey</material>
-    <mu1>0.9</mu1>
-    <mu2>0.9</mu2>
-    <kp>100000</kp>
-    <kd>100</kd>
-    <minDepth>0.00005</minDepth>
-    <maxVel>0.1</maxVel>
-    <maxContacts>3</maxContacts>
-  </gazebo>
-  <gazebo reference="roller_027_link">
-    <material>Gazebo/Grey</material>
-    <mu1>0.9</mu1>
-    <mu2>0.9</mu2>
-    <kp>100000</kp>
-    <kd>100</kd>
-    <minDepth>0.00005</minDepth>
-    <maxVel>0.1</maxVel>
-    <maxContacts>3</maxContacts>
-  </gazebo>
-  <gazebo reference="roller_028_link">
-    <material>Gazebo/Grey</material>
-    <mu1>0.9</mu1>
-    <mu2>0.9</mu2>
-    <kp>100000</kp>
-    <kd>100</kd>
-    <minDepth>0.00005</minDepth>
-    <maxVel>0.1</maxVel>
-    <maxContacts>3</maxContacts>
-  </gazebo>
-  <gazebo reference="roller_029_link">
-    <material>Gazebo/Grey</material>
-    <mu1>0.9</mu1>
-    <mu2>0.9</mu2>
-    <kp>100000</kp>
-    <kd>100</kd>
-    <minDepth>0.00005</minDepth>
-    <maxVel>0.1</maxVel>
-    <maxContacts>3</maxContacts>
-  </gazebo>
-  <gazebo reference="roller_030_link">
-    <material>Gazebo/Grey</material>
-    <mu1>0.9</mu1>
-    <mu2>0.9</mu2>
-    <kp>100000</kp>
-    <kd>100</kd>
-    <minDepth>0.00005</minDepth>
-    <maxVel>0.1</maxVel>
-    <maxContacts>3</maxContacts>
-  </gazebo>
-  <gazebo reference="roller_031_link">
-    <material>Gazebo/Grey</material>
-    <mu1>0.9</mu1>
-    <mu2>0.9</mu2>
-    <kp>100000</kp>
-    <kd>100</kd>
-    <minDepth>0.00005</minDepth>
-    <maxVel>0.1</maxVel>
-    <maxContacts>3</maxContacts>
-  </gazebo>
-  <gazebo reference="roller_032_link">
-    <material>Gazebo/Grey</material>
-    <mu1>0.9</mu1>
-    <mu2>0.9</mu2>
-    <kp>100000</kp>
-    <kd>100</kd>
-    <minDepth>0.00005</minDepth>
-    <maxVel>0.1</maxVel>
-    <maxContacts>3</maxContacts>
-  </gazebo>
-  <gazebo reference="roller_033_link">
-    <material>Gazebo/Grey</material>
-    <mu1>0.9</mu1>
-    <mu2>0.9</mu2>
-    <kp>100000</kp>
-    <kd>100</kd>
-    <minDepth>0.00005</minDepth>
-    <maxVel>0.1</maxVel>
-    <maxContacts>3</maxContacts>
-  </gazebo>
-  <gazebo reference="roller_034_link">
-    <material>Gazebo/Grey</material>
-    <mu1>0.9</mu1>
-    <mu2>0.9</mu2>
-    <kp>100000</kp>
-    <kd>100</kd>
-    <minDepth>0.00005</minDepth>
-    <maxVel>0.1</maxVel>
-    <maxContacts>3</maxContacts>
-  </gazebo>
-  <gazebo reference="roller_035_link">
-    <material>Gazebo/Grey</material>
-    <mu1>0.9</mu1>
-    <mu2>0.9</mu2>
-    <kp>100000</kp>
-    <kd>100</kd>
-    <minDepth>0.00005</minDepth>
-    <maxVel>0.1</maxVel>
-    <maxContacts>3</maxContacts>
-  </gazebo>
-  <gazebo reference="roller_036_link">
-    <material>Gazebo/Grey</material>
-    <mu1>0.9</mu1>
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
Commit message: gazebo and rviz

File: sentinel_ws/src/sentry_description/urdf/chassis.xacro (robot description, xacro)
@@ -31,6 +31,8 @@
        碰撞体是包住滚子的球，惯量按球近似，球心/质心用 CAD 的 com。 -->
   <xacro:macro name="cad_roller" params="id parent xyz axis com r i">
-    <link name="roller_${id}_link">
-      <xacro:cad_visual file="roller_${id}_link.stl"/>
+    <!-- Xacro 将 001 等参数解析为整数；显式补零以匹配 CAD 文件名。 -->
+    <xacro:property name="roller_name" value="${'roller_%03d' % int(id)}"/>
+    <link name="${roller_name}_link">
+      <xacro:cad_visual file="${roller_name}_link.stl"/>
       <inertial>
         <mass value="${roller_mass}"/>
@@ -45,7 +47,7 @@
       </collision>
     </link>
-    <joint name="roller_${id}_joint" type="continuous">
+    <joint name="${roller_name}_joint" type="continuous">
       <parent link="${parent}"/>
-      <child link="roller_${id}_link"/>
+      <child link="${roller_name}_link"/>
       <origin xyz="${xyz}"/>
       <axis xyz="${axis}"/>

File: sentinel_ws/src/sentry_sim/urdf/sentry_sim.urdf.xacro (robot description, xacro)
@@ -14,5 +14,5 @@
   <!-- 滚子接触参数：高刚度 + 软阻尼，压住全向轮打滑 -->
   <xacro:macro name="roller_surface" params="n">
-    <gazebo reference="roller_${n}_link">
+    <gazebo reference="roller_${'%03d' % int(n)}_link">
       <material>Gazebo/Grey</material>
       <mu1>0.9</mu1>
